File: projet/projet.kicad_sch (KiCad schematic)
At the start: 8 parts, among them J301 EMB_P3.81_1x02_VERTICAL, J302 EMB_P3.81_1x04_VERTICAL, U1 RASPBERRY_PI_PICO

Commit message: mise à jour du schematic avec les test points et ajout des TVS et inversion vcc gnd sur l'entrée
Parts:
- added D302, D303: TVS 5V, codium_Basics:SOD323_NP, symbol codium_Diodes:TVS_5V_BIDIR_SOD323
- added TP301: TestGND, symbol Connector:TestPoint
- added TP302: TestVCC, symbol Connector:TestPoint
- added TP303: TestCapteur, symbol Connector:TestPoint
- added TP304: TestLED, symbol Connector:TestPoint
Connections:
- net +5V: now also D301.1 (A1), J301.1 (Pin_1), D303.2 (A2), TP302.1; no longer D301.2 (A2), J301.2 (Pin_2)
- net GND: now also D301.2 (A2), J301.2 (Pin_2), U1.AGND, U1.GND2, U1.GND3, U1.GND4, U1.GND5, U1.GND6, U1.GND7, D302.2 (A2), D303.1 (A1), TP301.1; no longer D301.1 (A1), J301.1 (Pin_1)
- net lecteur_ir_13: now also U1.GP13, TP303.1
- net ruban_led_7: now also D302.1 (A1), TP304.1
Other:
- note added: "connecteur LED"
